File: kicad/midi2cv/trigout.sch (KiCad schematic (older format))
At the start: 26 parts, among them J14 Conn_01x08_Male, J15 Conn_01x08_Female, J16 P1, J17 P2, J18 P3, J19 P4, J20 P5, J21 P6, J22 P7, J23 P8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

Commit message: Create pcb.
Parts:
- removed J14: Conn_01x08_Male, Connector_PinSocket_2.54mm:PinSocket_1x08_P2.54mm_Vertical, symbol Connector:Conn_01x08_Male
- removed J15: Conn_01x08_Female, Connector_PinHeader_2.54mm:PinHeader_1x08_P2.54mm_Vertical, symbol Connector:Conn_01x08_Female
- added J14, J15: Conn_01x04_Male, Connector_PinSocket_2.54mm:PinSocket_1x04_P2.54mm_Vertical, symbol Connector:Conn_01x04_Male
- added J24, J25: Conn_01x04_Female, Connector_PinHeader_2.54mm:PinHeader_1x04_P2.54mm_Vertical, symbol Connector:Conn_01x04_Female
Connections:
- net at U6.1, U6.2 (-): now also J14.4 (Pin_4)
- net at U6.6 (-), U6.7: now also J14.3 (Pin_3)
- net at U6.8, U6.9 (-): now also J14.2 (Pin_2)
- net at U6.13 (-), U6.14: now also J14.1 (Pin_1)
- net at U8.1, U8.2 (-): now also J15.4 (Pin_4)
- net at U8.6 (-), U8.7: now also J15.3 (Pin_3)
- net at U8.8, U8.9 (-): now also J15.2 (Pin_2)
- net at U8.13 (-), U8.14: now also J15.1 (Pin_1)
- net at R8.1: now also J24.4 (Pin_4)
- net at R9.1: now also J24.3 (Pin_3)
- net at R10.1: now also J24.2 (Pin_2)
- net at R11.1: now also J24.1 (Pin_1)
- net at R12.1: now also J25.4 (Pin_4)
- net at R13.1: now also J25.3 (Pin_3)
- net at R14.1: now also J25.2 (Pin_2)
- net at R15.1: now also J25.1 (Pin_1)
Changed lines of the file:
@@
 NoConn ~ 8900 5850
 NoConn ~ 2850 4050
-$Comp
-L Connector:Conn_01x08_Male J14
-U 1 1 5CFF758B
-P 6600 3550
-F 0 "J14" H 6800 4050 50  0000 R CNN
-F 1 "Conn_01x08_Male" H 6800 3950 50  0000 R CNN
-F 2 "Connector_PinSocket_2.54mm:PinSocket_1x08_P2.54mm_Vertical" H 6600 3550 50  0001 C CNN
-F 3 "~" H 6600 3550 50  0001 C CNN
-	1    6600 3550
-	-1   0    0    1
-$EndComp
-$Comp
-L Connector:Conn_01x08_Female J15
-U 1 1 5CFF7824
-P 6800 3550
-F 0 "J15" H 6650 2900 50  0000 C CNN
-F 1 "Conn_01x08_Female" H 6950 3000 50  0000 C CNN
-F 2 "Connector_PinHeader_2.54mm:PinHeader_1x08_P2.54mm_Vertical" H 6800 3550 50  0001 C CNN
-F 3 "~" H 6800 3550 50  0001 C CNN
-	1    6800 3550
-	-1   0    0    1
-$EndComp
 Wire Wire Line
 	5450 3450 5450 3150
@@
 	1    0    0    -1
 $EndComp
+$Comp
+L Connector:Conn_01x04_Male J14
+U 1 1 5CE478A9
+P 6600 3350
+F 0 "J14" H 6700 2900 50  0000 R CNN
+F 1 "Conn_01x04_Male" H 7250 3000 50  0000 R CNN
+F 2 "Connector_PinSocket_2.54mm:PinSocket_1x04_P2.54mm_Vertical" H 6600 3350 50  0001 C CNN
+F 3 "~" H 6600 3350 50  0001 C CNN
+	1    6600 3350
+	-1   0    0    1
+$EndComp
+$Comp
+L Connector:Conn_01x04_Male J15
+U 1 1 5CE47981
+P 6600 3750
+F 0 "J15" H 6700 4050 50  0000 R CNN
+F 1 "Conn_01x04_Male" H 7250 3950 50  0000 R CNN
+F 2 "Connector_PinSocket_2.54mm:PinSocket_1x04_P2.54mm_Vertical" H 6600 3750 50  0001 C CNN
+F 3 "~" H 6600 3750 50  0001 C CNN
+	1    6600 3750
+	-1   0    0    1
+$EndComp
+$Comp
+L Connector:Conn_01x04_Female J24
+U 1 1 5CE47D41
+P 6800 3350
+F 0 "J24" H 6800 2900 50  0000 C CNN
+F 1 "Conn_01x04_Female" H 6500 3000 50  0000 C CNN
+F 2 "Connector_PinHeader_2.54mm:PinHeader_1x04_P2.54mm_Vertical" H 6800 3350 50  0001 C CNN
+F 3 "~" H 6800 3350 50  0001 C CNN
+	1    6800 3350
+	-1   0    0    1
+$EndComp
+$Comp
+L Connector:Conn_01x04_Female J25
+U 1 1 5CE47E01
+P 6800 3750
+F 0 "J25" H 6800 4050 50  0000 C CNN
+F 1 "Conn_01x04_Female" H 6500 3950 50  0000 C CNN
+F 2 "Connector_PinHeader_2.54mm:PinHeader_1x04_P2.54mm_Vertical" H 6800 3750 50  0001 C CNN
+F 3 "~" H 6800 3750 50  0001 C CNN
+	1    6800 3750
+	-1   0    0    1
+$EndComp
 $EndSCHEMATC
